File: humidity.brd (EAGLE design)
At the start: 34 x 62.2 mm, 9 parts

Commit message: upravena DPS
Parts:
- moved NAPAJENI 2.54 mm to (10.2, 57.1)
- moved R1 1.27 mm to (29.2, 53.3)
Routing:
- net +3V3: track 115.6 -> 122.9 mm
- net N$13: track 7.88 -> 6.61 mm
- net N$15: track 25.7 -> 24.5 mm
- net GND: track 84.0 -> 84.8 mm

Commit message: DPS
Connections:
- net GND: now also U$1.GPIO15
Routing:
- net GND: track 84.8 -> 106.4 mm
Changed lines of the file:
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@@
 <?xml version="1.0" encoding="utf-8"?>
 <!DOCTYPE eagle SYSTEM "eagle.dtd">
-<eagle version="6.5.0">
+<eagle version="7.3.0">
 <drawing>
 <settings>
@@
 <pass name="Default">
 <param name="RoutingGrid" value="50mil"/>
+<param name="AutoGrid" value="1"/>
+<param name="Efforts" value="0"/>
+<param name="TopRouterVariant" value="1"/>
 <param name="tpViaShape" value="round"/>
 <param name="PrefDir.1" value="|"/>
@@
 <wire x1="3.81" y1="49.53" x2="3.81" y2="46.99" width="1.016" layer="16"/>
 <wire x1="7.62" y1="5.08" x2="10.16" y2="5.08" width="1.016" layer="16"/>
-<wire x1="10.16" y1="5.08" x2="10.16" y2="21.59" width="1.016" layer="16"/>
+<wire x1="10.16" y1="5.08" x2="10.16" y2="8.89" width="1.016" layer="16"/>
+<wire x1="10.16" y1="8.89" x2="10.16" y2="21.59" width="1.016" layer="16"/>
 <wire x1="10.16" y1="21.59" x2="10.16" y2="33.02" width="1.016" layer="16"/>
 <wire x1="10.16" y1="33.02" x2="1.27" y2="33.02" width="0.4064" layer="16"/>
@@
 <wire x1="3.81" y1="49.53" x2="3.81" y2="52.705" width="1.016" layer="16"/>
 <wire x1="3.81" y1="52.705" x2="7.62" y2="56.515" width="1.016" layer="16"/>
+<contactref element="U$1" pad="GPIO15"/>
+<wire x1="3.81" y1="8.89" x2="10.16" y2="8.89" width="0.4064" layer="16"/>
+<wire x1="3.81" y1="8.89" x2="3.81" y2="24.13" width="1.016" layer="16"/>
 </signal>
 <signal name="N$2">
